Commit message: Task 8.1: Sabotaged odometry, laser scanner, SLAM mapping, saved map

File: urdf/differential_robot_task8.urdf (robot description, URDF)
Before this commit: robot diff_drive_robot, 5 links, 4 joints
Links:
- added link laser_link, mass 0.050; collision cylinder length=0.02 radius=0.03; visual cylinder length=0.02 radius=0.03
Joints:
- added joint base_to_laser: type fixed, parent base_link, child laser_link, origin xyz=0 0 0.06
